File: Students/Cooper95/KiCad/Project3/Project3.kicad_pcb (KiCad board)
At the start: 2 copper layers, 17 parts, among them CON1 BARREL_JACK, P1 CONN_01X04, P2 CONN_01X17, Q1 MMBT3906, Q2 MMBT3906, SW1 Switch_SPDT_x2, SW2 Switch_SPDT_x2, U1 Teensy_3.1, U2 LM7805CT

Commit message: Project 3 PCB
Parts:
- Q1, Q2: footprint SOT-23 -> Power_Integrations:TO-220
- SW1: footprint CustomSwitch:SPDT-ThroughHole -> SPDT-ThroughHole
- moved SW1 51.7 mm to (115.6, 113.0)
- moved SW2 46.6 mm to (129.5, 113.0)
- moved D3 37.1 mm to (190.5, 91.4), turned to 180 degrees
- moved P1 34.4 mm to (157.5, 91.4), turned to 270 degrees
- moved R4 32.8 mm to (149.9, 110.5)
- moved D1 31.0 mm to (118.1, 91.4)
- moved R1 29.0 mm to (149.9, 116.8)
- moved U2 26.9 mm to (128.3, 101.6), turned to 270 degrees
- moved R2 26.0 mm to (168.9, 88.9), turned to 180 degrees
- moved R3 23.8 mm to (168.9, 92.7), turned to 180 degrees
- moved D4 23.3 mm to (134.6, 91.4)
- moved D2 21.0 mm to (182.9, 91.4), turned to 180 degrees
- moved Q2 15.7 mm to (148.6, 101.6), turned to 270 degrees
- moved U1 8.89 mm to (190.5, 99.1)
- moved Q1 6.84 mm to (138.4, 101.6), turned to 270 degrees
Connections:
- U1 pad 3: /Pump2PWM -> /Pump1PWM
- U1 pad 4: /Pump1PWM -> /Pump2PWM
Routing:
- net +5V: track 0.00 -> 147.0 mm
- net +12V: track 0.00 -> 93.3 mm
- net /FlowSens: track 0.00 -> 49.4 mm
- net Net-(D1-Pad2): track 0.00 -> 41.4 mm, vias 0 -> 2
- net /Pump1PWM: track 0.00 -> 36.8 mm
- net Net-(D4-Pad2): track 0.00 -> 36.0 mm
- net /Pump2PWM: track 0.00 -> 30.1 mm
- net Earth: track 0.00 -> 25.1 mm, vias 0 -> 3
- net /SCLK: track 0.00 -> 25.0 mm
- net Net-(Q1-Pad1): track 0.00 -> 21.9 mm
- net /SDA: track 0.00 -> 21.7 mm
- net /BT_TX: track 0.00 -> 19.9 mm
- net /BT_RX: track 0.00 -> 19.1 mm
- net Net-(D3-Pad2): track 0.00 -> 16.6 mm
- net /TeensyPWR: track 0.00 -> 16.3 mm
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- added copper zone on B.Cu, net Earth
- added copper zone on F.Cu, net Earth
Other:
- board outline added: 88.9 x 43.2 mm
- net class Default: clearance 0.2 -> 0.508; trace_width 0.25 -> 0.508; via_dia 0.6 -> 0.508; via_drill 0.4 -> 0.4064
- net class Power added: clearance 0.508, trace_width 1.016, via_dia 0.508, via_drill 0.4064
- rule trace_clearance: 0.2 -> 0.508
- rule trace_min: 0.2 -> 0.508
- rule via_min_drill: 0.3 -> 0.4064
- rule via_min_size: 0.4 -> 0.508

Commit message: Finished project 3 board and BOM
Parts:
- added SW3: SW_PUSH, Buttons_Switches_ThroughHole:SW_PUSH_SMALL, F.Cu at (139.7, 111.8)
- moved SW2 3.81 mm to (125.7, 113.0)
- moved SW1 2.54 mm to (113.0, 113.0)
Connections:
- U1 pad 26: +5V -> Net-(SW3-Pad1)
Routing:
- net Net-(SW3-Pad1): track 0.00 -> 61.6 mm
- net +5V: track 147.0 -> 122.3 mm
- net Net-(D1-Pad2): track 41.4 -> 47.0 mm
- net Net-(D4-Pad2): track 36.0 -> 39.8 mm
- net Earth: track 25.1 -> 26.9 mm
- net /Pump2GND: track 14.3 -> 12.7 mm
- net /Pump1GND: track 12.7 -> 13.8 mm
